Commit message: Replace MoveIt IK with geometric IK solver, fix TCP offset, add camera pose publisher
- Fix TCP offset to official value (-0.0079, -0.000218, -0.0981274) in URDF and compute_workspace.py
- Add analytical geometric_ik() solver: 0.3mm accuracy, 84µs/call (243x faster than FK sweep)
- Simplify control_gui.py IK pipeline: geometric IK for grasps, MoveIt fallback for non-grasp moves
- Remove _find_best_wrist_roll (360-step FK sweep) and _correct_grasp_wrist_flex (replaced by analytical formulas)
- Add calibrate_ik.py to auto-derive all IK constants from FK chain (replaces manual derivation)
- Add camera_pose_publisher node (TF2 base->camera_link) to control and gazebo launches
- Fix USD base frame to match URDF (was 16.8mm X offset)
- Regenerate workspace bounds with corrected TCP

File: vla_SO-ARM101/src/so_arm101_description/urdf/so_arm101.urdf (robot description, URDF)
Before this commit: robot so_arm101, 10 links, 9 joints
Links:
- added link tcp_link
Joints:
- added joint tcp_joint: type fixed, parent gripper, child tcp_link, origin xyz=-0.0079 -0.000218121 -0.0981274 rpy=0 3.14159 0
- joint elbow_flex: limit lower=-1.74533 upper=1.5708 effort=10 velocity=10 -> lower=-1.69 upper=1.69 effort=10 velocity=10
- joint shoulder_pan: origin xyz=0 -0.0220095 0.0648007 rpy=-3.14159 6.03684e-16 1.5708 -> xyz=0.0388353 -8.97657e-09 0.0624 rpy=3.14159 4.18253e-17 -3.14159
- joint wrist_roll: limit lower=-2.79253 upper=2.79253 effort=10 velocity=10 -> lower=-2.74385 upper=2.84121 effort=10 velocity=10; origin xyz=0 -0.0611 0.0181 rpy=1.5708 -9.38083e-08 3.14159 -> xyz=0 -0.0611 0.0181 rpy=1.5708 0.0486795 3.14159
