Commit message: Fix base link offset and rename joints to LeRobot SO-101 spec
Base link visual/collision meshes from onshape-to-robot export were
offset ~2.1cm in X and hovering ~3cm above the link origin. Shifted
all base mesh origins, inertial, and base-to-shoulder joint to center
and ground the robot at the origin.

Renamed all joint names across the codebase to match the official
LeRobot SO-101 specification:
  Rotation    -> shoulder_pan
  Pitch       -> shoulder_lift
  Elbow       -> elbow_flex
  Wrist_Pitch -> wrist_flex
  Wrist_Roll  -> wrist_roll
  Jaw         -> gripper

File: vla_SO-ARM101/src/so_arm101_description/urdf/so_arm101.gazebo.xacro (robot description, xacro)
@@ -13,30 +13,30 @@
       <plugin>gz_ros2_control/GazeboSimSystem</plugin>
     </hardware>
-    <joint name="Rotation">
+    <joint name="shoulder_pan">
       <command_interface name="position"/>
       <state_interface name="position"/>
       <state_interface name="velocity"/>
     </joint>
-    <joint name="Pitch">
+    <joint name="shoulder_lift">
       <command_interface name="position"/>
       <state_interface name="position"/>
       <state_interface name="velocity"/>
     </joint>
-    <joint name="Elbow">
+    <joint name="elbow_flex">
       <command_interface name="position"/>
       <state_interface name="position"/>
       <state_interface name="velocity"/>
     </joint>
-    <joint name="Wrist_Pitch">
+    <joint name="wrist_flex">
       <command_interface name="position"/>
       <state_interface name="position"/>
       <state_interface name="velocity"/>
     </joint>
-    <joint name="Wrist_Roll">
+    <joint name="wrist_roll">
       <command_interface name="position"/>
       <state_interface name="position"/>
       <state_interface name="velocity"/>
     </joint>
-    <joint name="Jaw">
+    <joint name="gripper">
       <command_interface name="position"/>
       <state_interface name="position"/>

File: vla_SO-ARM101/src/so_arm101_description/urdf/so_arm101.urdf (robot description, URDF)
Before this commit: robot so_arm101, 7 links, 6 joints
Joints:
- removed joint Elbow
- removed joint Jaw
- removed joint Pitch
- removed joint Rotation
- removed joint Wrist_Pitch
- removed joint Wrist_Roll
- added joint elbow_flex: type revolute, parent upper_arm, child lower_arm, origin xyz=-0.11257 -0.028 2.46331e-16 rpy=-1.22818e-15 5.75928e-16 1.5708, axis 0 0 1, limit lower=-1.74533 upper=1.5708 effort=10 velocity=10
- added joint gripper: type revolute, parent gripper, child jaw, origin xyz=0.0202 0.0188 -0.0234 rpy=1.5708 -5.14108e-17 -1.38655e-14, axis 0 0 1, limit lower=-0.174533 upper=1.74533 effort=10 velocity=10
- added joint shoulder_lift: type revolute, parent shoulder, child upper_arm, origin xyz=-0.0303992 -0.0182778 -0.0542 rpy=-1.5708 -1.5708 0, axis 0 0 1, limit lower=-1.74533 upper=1.74533 effort=10 velocity=10
- added joint shoulder_pan: type revolute, parent base, child shoulder, origin xyz=0 -0.0220095 0.0648007 rpy=-3.14159 6.03684e-16 1.5708, axis 0 0 1, limit lower=-1.91986 upper=1.91986 effort=10 velocity=10
- added joint wrist_flex: type revolute, parent lower_arm, child wrist, origin xyz=-0.1349 0.0052 1.65232e-16 rpy=3.2474e-15 2.86219e-15 -1.5708, axis 0 0 1, limit lower=-1.65806 upper=1.65806 effort=10 velocity=10
- added joint wrist_roll: type revolute, parent wrist, child gripper, origin xyz=0 -0.0611 0.0181 rpy=1.5708 -9.38083e-08 3.14159, axis 0 0 1, limit lower=-2.79253 upper=2.79253 effort=10 velocity=10

File: vla_SO-ARM101/src/so_arm101_moveit_config/config/so_arm101.ros2_control.xacro (robot description, xacro)
@@ -9,43 +9,43 @@
                 <plugin>mock_components/GenericSystem</plugin>
             </hardware>
-            <joint name="Rotation">
+            <joint name="shoulder_pan">
                 <command_interface name="position"/>
                 <state_interface name="position">
-                  <param name="initial_value">${initial_positions['Rotation']}</param>
+                  <param name="initial_value">${initial_positions['shoulder_pan']}</param>
                 </state_interface>
                 <state_interface name="velocity"/>
             </joint>
-            <joint name="Pitch">
+            <joint name="shoulder_lift">
                 <command_interface name="position"/>
                 <state_interface name="position">
-                  <param name="initial_value">${initial_positions['Pitch']}</param>
+                  <param name="initial_value">${initial_positions['shoulder_lift']}</param>
                 </state_interface>
                 <state_interface name="velocity"/>
             </joint>
-            <joint name="Elbow">
+            <joint name="elbow_flex">
                 <command_interface name="position"/>
                 <state_interface name="position">
-                  <param name="initial_value">${initial_positions['Elbow']}</param>
+                  <param name="initial_value">${initial_positions['elbow_flex']}</param>
                 </state_interface>
                 <state_interface name="velocity"/>
             </joint>
-            <joint name="Wrist_Pitch">
+            <joint name="wrist_flex">
                 <command_interface name="position"/>
                 <state_interface name="position">
-                  <param name="initial_value">${initial_positions['Wrist_Pitch']}</param>
+                  <param name="initial_value">${initial_positions['wrist_flex']}</param>
                 </state_interface>
                 <state_interface name="velocity"/>
             </joint>
-            <joint name="Wrist_Roll">
+            <joint name="wrist_roll">
                 <command_interface name="position"/>
                 <state_interface name="position">
-                  <param name="initial_value">${initial_positions['Wrist_Roll']}</param>
+                  <param name="initial_value">${initial_positions['wrist_roll']}</param>
                 </state_interface>
                 <state_interface name="velocity"/>
             </joint>
-            <joint name="Jaw">
+            <joint name="gripper">
                 <command_interface name="position"/>
                 <state_interface name="position">
-                  <param name="initial_value">${initial_positions['Jaw']}</param>
+                  <param name="initial_value">${initial_positions['gripper']}</param>
                 </state_interface>
                 <state_interface name="velocity"/>

Commit message: Add camera mount with Gazebo wrist camera and fix gripper joint naming
- Add camera_link and camera_optical_frame to URDF at lens center
  (centroid of 4 camera screw holes M0-M3 on the mount STL)
- Add Ignition Gazebo camera sensor on camera_link (640x480, 30Hz)
- Bridge wrist_camera image and camera_info topics via ros_gz_bridge
- Rename joint "gripper" to "gripper_joint" to fix SDF name collision
  (Gazebo SDF requires unique names across links and joints)
- Update joint name in all configs: SRDF, ros2_controllers, ros2_control
  xacro, initial_positions, control_gui, servo_driver, joint_state_reader
- Add disable_collisions entries for camera_mount vs gripper/jaw/wrist

File: vla_SO-ARM101/src/so_arm101_description/urdf/so_arm101.gazebo.xacro (robot description, xacro)
@@ -38,5 +38,5 @@
       <state_interface name="velocity"/>
     </joint>
-    <joint name="gripper">
+    <joint name="gripper_joint">
       <command_interface name="position"/>
       <state_interface name="position"/>
@@ -93,3 +93,30 @@
     </material>
   </gazebo>
+  <gazebo reference="camera_mount">
+    <material>
+      <ambient>1.0 0.82 0.12 1</ambient>
+      <diffuse>1.0 0.82 0.12 1</diffuse>
+    </material>
+  </gazebo>
+  <!-- Wrist camera sensor (Ignition Gazebo) -->
+  <gazebo reference="camera_link">
+    <sensor name="wrist_camera" type="camera">
+      <camera>
+        <horizontal_fov>1.047</horizontal_fov>
+        <image>
+          <width>640</width>
+          <height>480</height>
+          <format>R8G8B8</format>
+        </image>
+        <clip>
+          <near>0.01</near>
+          <far>100</far>
+        </clip>
+      </camera>
+      <always_on>1</always_on>
+      <update_rate>30</update_rate>
+      <visualize>true</visualize>
+      <topic>wrist_camera</topic>
+    </sensor>
+  </gazebo>
 </robot>

File: vla_SO-ARM101/src/so_arm101_description/urdf/so_arm101.urdf (robot description, URDF)
Before this commit: robot so_arm101, 7 links, 6 joints
Links:
- added link camera_link
- added link camera_mount; collision mesh filename=package://so_arm101_description/meshes/obj_3_SO-ARM101_came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 scale=0.001 0.001 0.001; visual mesh filename=package://so_arm101_description/meshes/obj_3_SO-ARM101_came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 scale=0.001 0.001 0.001
- added link camera_optical_frame
Joints:
- removed joint gripper
- added joint camera_link_joint: type fixed, parent camera_mount, child camera_link, origin xyz=-0.010350 0.023428 0.004830 rpy=0 0 1.5708
- added joint camera_mount_joint: type fixed, parent gripper, child camera_mount, origin xyz=0.002359 0.049561 -0.011838 rpy=-2.956686 -0.384393 -2.034078
- added joint camera_optical_joint: type fixed, parent camera_link, child camera_optical_frame, origin xyz=0 0 0 rpy=-1.5708 0 -1.5708
- added joint gripper_joint: type revolute, parent gripper, child jaw, origin xyz=0.0202 0.0188 -0.0234 rpy=1.5708 -5.14108e-17 -1.38655e-14, axis 0 0 1, limit lower=-0.174533 upper=1.74533 effort=10 velocity=10

File: vla_SO-ARM101/src/so_arm101_moveit_config/config/so_arm101.ros2_control.xacro (robot description, xacro)
@@ -44,8 +44,8 @@
                 <state_interface name="velocity"/>
             </joint>
-            <joint name="gripper">
+            <joint name="gripper_joint">
                 <command_interface name="position"/>
                 <state_interface name="position">
-                  <param name="initial_value">${initial_positions['gripper']}</param>
+                  <param name="initial_value">${initial_positions['gripper_joint']}</param>
                 </state_interface>
                 <state_interface name="velocity"/>

Commit message: Add USB camera mesh aligned to camera mount via hole detection
- Detect mounting holes in both camera mount (4x r=1mm, 27mm square)
  and ELP USB camera (4x corner holes, 29mm square) using trimesh
- Compute rigid alignment via Kabsch algorithm (RMSD 1.5mm)
- Add usb_camera link with visual/collision mesh to URDF
- Fix camera_link to ROS convention (X-forward) as child of usb_camera
- Fix camera_optical_frame to OpenCV convention (X-right, Y-down, Z-forward)
- Update Gazebo sensor to reference usb_camera with ignition_frame_id

File: vla_SO-ARM101/src/so_arm101_description/urdf/so_arm101.gazebo.xacro (robot description, xacro)
@@ -99,8 +99,19 @@
     </material>
   </gazebo>
+  <gazebo reference="usb_camera">
+    <material>
+      <ambient>0.1 0.1 0.1 1</ambient>
+      <diffuse>0.1 0.1 0.1 1</diffuse>
+    </material>
+  </gazebo>
   <!-- Wrist camera sensor (Ignition Gazebo) -->
-  <gazebo reference="camera_link">
+  <gazebo reference="usb_camera">
     <sensor name="wrist_camera" type="camera">
-      <camera>
+      <pose>0 0.0029 0 0 1.5708 0</pose>
+      <always_on>1</always_on>
+      <update_rate>30</update_rate>
+      <visualize>true</visualize>
+      <ignition_frame_id>camera_link</ignition_frame_id>
+      <camera name="wrist_camera">
         <horizontal_fov>1.047</horizontal_fov>
         <image>
@@ -111,11 +122,9 @@
         <clip>
           <near>0.01</near>
-          <far>100</far>
+          <far>10.0</far>
         </clip>
       </camera>
-      <always_on>1</always_on>
-      <update_rate>30</update_rate>
-      <visualize>true</visualize>
       <topic>wrist_camera</topic>
+      <camera_info_topic>wrist_camera/camera_info</camera_info_topic>
     </sensor>
   </gazebo>

File: vla_SO-ARM101/src/so_arm101_description/urdf/so_arm101.urdf (robot description, URDF)
Before this commit: robot so_arm101, 11 links, 10 joints
Links:
- added link usb_camera; collision mesh filename=package://so_arm101_description/meshes/usb_cam_elp.stl scale=0.001 0.001 0.001; visual mesh filename=package://so_arm101_description/meshes/usb_cam_elp.stl scale=0.001 0.001 0.001
Joints:
- added joint usb_camera_joint: type fixed, parent camera_mount, child usb_camera, origin xyz=-0.010340 0.004827 -0.019687 rpy=1.570625 0.000515 2.705234
- joint camera_link_joint: origin xyz=-0.010350 0.023428 0.004830 rpy=0 0 1.5708 -> xyz=0 0.0029 0 rpy=0 0 -1.5708; parent camera_mount -> usb_camera

Commit message: Fix wrist camera sensor pose and FOV from mesh-derived lens position
- Set sensor pose Y to 0.0139m (lens center measured from usb_cam_elp.stl
  barrel face, was 0.0029m which placed camera inside mount ring)
- Match camera_link_joint translation for TF consistency
- Widen FOV from 60° to 100° to match OV9732 USB camera specs

File: vla_SO-ARM101/src/so_arm101_description/urdf/so_arm101.gazebo.xacro (robot description, xacro)
@@ -108,5 +108,5 @@
   <gazebo reference="usb_camera">
     <sensor name="wrist_camera" type="camera">
-      <pose>0 0.0029 0 1.5708 0 1.5708</pose>
+      <pose>0 0.0139 0 1.5708 0 1.5708</pose>
       <always_on>1</always_on>
       <update_rate>30</update_rate>
@@ -114,5 +114,5 @@
       <ignition_frame_id>camera_link</ignition_frame_id>
       <camera name="wrist_camera">
-        <horizontal_fov>1.047</horizontal_fov>
+        <horizontal_fov>1.7453</horizontal_fov>
         <image>
           <width>1280</width>

File: vla_SO-ARM101/src/so_arm101_description/urdf/so_arm101.urdf (robot description, URDF)
Before this commit: robot so_arm101, 12 links, 11 joints
Joints:
- joint camera_link_joint: origin xyz=0 0.0029 0 rpy=0 0 -1.5708 -> xyz=0 0.0139 0 rpy=0 0 -1.5708

Commit message: Add YOLOE detection verification for SO-ARM101
- verify_detections.py: compares YOLOE detections against Gazebo GT
  using world->base TF, 5s periodic reports, 50mm pass threshold
- Add verify_detections console entry point to setup.py

File: vla_SO-ARM101/src/so_arm101_description/urdf/so_arm101.gazebo.xacro (robot description, xacro)
@@ -106,7 +106,7 @@
   </gazebo>
   <!-- Wrist camera sensor (Ignition Gazebo) -->
-  <gazebo reference="usb_camera">
+  <gazebo reference="camera_link">
     <sensor name="wrist_camera" type="camera">
-      <pose>0 0.0139 0 1.5708 0 1.5708</pose>
+      <pose>0 0 0 0 0 0</pose>
       <always_on>1</always_on>
       <update_rate>30</update_rate>

File: vla_SO-ARM101/src/so_arm101_description/urdf/so_arm101.urdf (robot description, URDF)
Before this commit: robot so_arm101, 12 links, 11 joints
Joints:
- joint camera_link_joint: origin xyz=0 0.0139 0 rpy=0 0 -1.5708 -> xyz=0 0.0139 0 rpy=1.5708 0 1.5708

Commit message: feat(sim): add top_camera SDF sensor to so_arm101.gazebo.xacro
Phase 2, REQ OBS-03. Adds a second camera sensor to the Gazebo scene to
match the real SO-101 dataset's two-camera schema (wrist + top).

- New top_camera_link: fixed link 60cm above world origin
- New top_camera_joint: fixed parent=world, child=top_camera_link,
  origin xyz='0 0 0.6' rpy='0 1.5708 0' (optical axis pointing -Z)
- New <sensor name='top_camera' type='camera'>: 640x480 @ 30fps R8G8B8,
  horizontal_fov 1.2 rad, near 0.05 / far 5.0
- Publishes to Gazebo topics 'top_camera' and 'top_camera/camera_info'

Resolution matches the RealSense top camera used in the real flow
(see vla_SO-ARM101/docs/LEROBOT_GUIDE.md). Bridge config in
so_arm101_control/launch/gazebo.launch.py committed separately.

File: vla_SO-ARM101/src/so_arm101_description/urdf/so_arm101.gazebo.xacro (robot description, xacro)
@@ -129,3 +129,46 @@
     </sensor>
   </gazebo>
+  <!-- Top camera (tabletop top-down view for pick-and-place datasets).
+       Resolution 640x480 @ 30 fps R8G8B8 to match the real-flow RealSense top
+       camera (see LEROBOT_GUIDE.md). Mounted to a fixed top_camera_link 60 cm
+       above world origin, rotated so the optical axis points -Z (down). -->
+  <link name="top_camera_link">
+    <inertial>
+      <mass value="0.01"/>
+      <inertia ixx="1e-5" ixy="0" ixz="0" iyy="1e-5" iyz="0" izz="1e-5"/>
+    </inertial>
+    <visual>
+      <geometry><box size="0.04 0.04 0.02"/></geometry>
+      <material name="top_camera_black"><color rgba="0.1 0.1 0.1 1"/></material>
+    </visual>
+  </link>
+  <joint name="top_camera_joint" type="fixed">
+    <parent link="world"/>
+    <child link="top_camera_link"/>
+    <!-- 60 cm above origin; rpy rotates camera +X (image forward) to -Z world. -->
+    <origin xyz="0 0 0.6" rpy="0 1.5708 0"/>
+  </joint>
+  <gazebo reference="top_camera_link">
+    <sensor name="top_camera" type="camera">
+      <pose>0 0 0 0 0 0</pose>
+      <always_on>1</always_on>
+      <update_rate>30</update_rate>
+      <visualize>true</visualize>
+      <ignition_frame_id>top_camera_link</ignition_frame_id>
+      <camera name="top_camera">
+        <horizontal_fov>1.2</horizontal_fov>
+        <image>
+          <width>640</width>
+          <height>480</height>
+          <format>R8G8B8</format>
+        </image>
+        <clip>
+          <near>0.05</near>
+          <far>5.0</far>
+        </clip>
+      </camera>
+      <topic>top_camera</topic>
+      <camera_info_topic>top_camera/camera_info</camera_info_topic>
+    </sensor>
+  </gazebo>
 </robot>

Commit message: fix(sim): wrist camera — reparent to usb_camera + drop to 640x480
Gazebo Harmonic's Ogre2 silently refuses to create a render context
for a camera sensor attached to a link with no <visual>/<collision>.
camera_link was an empty URDF convention frame
(<link name="camera_link" />) — purely for ROS X-forward/Y-left/Z-up
transforms — so the <sensor> registered on the gz bus but produced 0
frames on the ROS2 /wrist_camera topic.

Reparented the <gazebo reference="..."> block from camera_link to
usb_camera (which has mesh geometry: meshes/usb_cam_elp.stl). The
URDF transform usb_camera -> camera_link (xyz="0 0.0139 0"
rpy="1.5708 0 1.5708") is folded into the sensor <pose> so the
effective optical axis sits exactly where it used to; verified
visually via side-by-side PNG snapshot of both topics. Kept
ignition_frame_id=camera_link so downstream Image messages carry
the original frame_id.

Dropped resolution 1280x720 -> 640x480 — matches the real RealSense
wrist view spec from LEROBOT_GUIDE.md, keeps macOS Ogre2 render rate
in the recording-usable range (>10 Hz; 1280x720 capped at ~0.5 Hz
on this Mac).

Dual-camera checkpoint through the Phase 3 so101_ros2 plugin:
20 observations clean, both cameras (480, 640, 3) uint8.

Runbook changelog entry added. Lerobot submodule pointer bumped to
e38a9c65 (planning doc refresh).

File: vla_SO-ARM101/src/so_arm101_description/urdf/so_arm101.gazebo.xacro (robot description, xacro)
@@ -105,8 +105,14 @@
     </material>
   </gazebo>
-  <!-- Wrist camera sensor (Ignition Gazebo) -->
-  <gazebo reference="camera_link">
+  <!-- Wrist camera. Re-parented from `camera_link` to `usb_camera` because
+       Gazebo Harmonic's Ogre2 won't create a render context for a sensor on
+       a geometry-less link (camera_link is a bare ROS-convention frame — no
+       <visual>/<collision>). The URDF transform from usb_camera to
+       camera_link (xyz="0 0.0139 0" rpy="1.5708 0 1.5708") is folded into
+       this sensor's <pose>. `ignition_frame_id` stays `camera_link` so
+       downstream /wrist_camera Image messages carry the original frame_id. -->
+  <gazebo reference="usb_camera">
     <sensor name="wrist_camera" type="camera">
-      <pose>0 0 0 0 0 0</pose>
+      <pose>0 0.0139 0 1.5708 0 1.5708</pose>
       <always_on>1</always_on>
       <update_rate>30</update_rate>
@@ -116,6 +122,9 @@
         <horizontal_fov>1.7453</horizontal_fov>
         <image>
-          <width>1280</width>
-          <height>720</height>
+          <!-- 640x480 matches the real RealSense wrist view and keeps macOS
+               Ogre2 render rate above 10 Hz. Raise to 1280x720 only if a
+               downstream recording needs it and you're OK with ~0.5 Hz. -->
+          <width>640</width>
+          <height>480</height>
           <format>R8G8B8</format>
         </image>
